Commit message: adding modified file for jbot6

File: lidarbot_description/urdf/camera.xacro (robot description, xacro)
@@ -4,5 +4,5 @@
   <link name="camera_link">
     <visual>
-      <origin xyz="-0.0115 0.0125 0.0052" rpy="${pi/2} ${pi} ${pi/2}"/>
+      <origin xyz="-0.140 0.0 0.117" rpy="${pi/2} ${pi} ${pi/2}"/>
       <geometry>
         <mesh filename="package://lidarbot_description/meshes/rpi_camera.dae"/>
@@ -13,5 +13,5 @@
     <parent link="base_link"/>
     <child link="camera_link"/>
-    <origin xyz="-0.15 0 0.28" rpy="0 0 0"/>
+    <origin xyz="0.140 0.0 0.117" rpy="0 0 0"/>
   </joint>
   <link name="camera_link_optical"></link>

File: lidarbot_description/urdf/gazebo_control.xacro (robot description, xacro)
@@ -6,6 +6,6 @@
             <left_joint>left_wheel_joint</left_joint>
             <right_joint>right_wheel_joint</right_joint>
-            <wheel_separation>0.233</wheel_separation>
-            <wheel_diameter>0.10</wheel_diameter>
+            <wheel_separation>0.300</wheel_separation>
+            <wheel_diameter>0.130</wheel_diameter>
             <!-- Limits (can be adjusted later on)-->
             <max_wheel_torque>20</max_wheel_torque>

File: lidarbot_description/urdf/imu.xacro (robot description, xacro)
@@ -12,5 +12,5 @@
     <parent link="base_link"/>
     <child link="imu_link"/>
-    <origin xyz="0.045 0 0.0175" rpy="0 0 0"/>
+    <origin xyz="0 0 0.010" rpy="0 0 0"/>
   </joint>
  <gazebo reference="imu_link">

File: lidarbot_description/urdf/lidar.xacro (robot description, xacro)
@@ -3,5 +3,5 @@
     <link name="lidar_link">
         <visual>
-            <origin xyz="0 -0.0009 -0.011" rpy="0 0 0"/>
+            <origin xyz="0 0 0" rpy="0 0 0"/>
             <geometry>
                 <mesh filename="package://lidarbot_description/meshes/rplidar_top.dae"/>
@@ -9,5 +9,5 @@
         </visual>
         <collision>
-            <origin xyz="0 -0.0028 0" rpy="0 0 0"/>
+            <origin xyz="0 0 0" rpy="0 0 0"/>
             <geometry>
                 <cylinder radius="0.037" length="0.021"/>
@@ -21,5 +21,5 @@
         <parent link="base_link"/>
         <child link="lidar_link"/>
-        <origin xyz="0 0 0.145" rpy="0 0 ${-pi/2}"/>
+        <origin xyz="0 0 0.180" rpy="0 0 ${-pi/2}"/>
         <axis xyz="0 0 1"/>
     </joint>
@@ -39,5 +39,5 @@
                 </scan>
                 <range>
-                    <min>0.15</min>
+                    <min>0.2</min>
                     <max>6.0</max>
                     <!-- <max>12.0</max> -->

File: lidarbot_description/urdf/lidarbot_core.xacro (robot description, xacro)
@@ -2,14 +2,14 @@
 <robot xmlns:xacro="http://www.ros.org/wiki/xacro" >
     <xacro:include filename="inertial_macros.xacro"/>
-    <xacro:property name="chassis_length" value="0.250"/>
-    <xacro:property name="chassis_width" value="0.147"/>
-    <xacro:property name="chassis_height" value="0.065"/>
+    <xacro:property name="chassis_length" value="0.280"/>
+    <xacro:property name="chassis_width" value="0.208"/>
+    <xacro:property name="chassis_height" value="0.375"/>
     <xacro:property name="chassis_mass" value="1.0"/>
-    <xacro:property name="wheel_radius" value="0.05"/>
-    <xacro:property name="wheel_thickness" value="0.040"/>
+    <xacro:property name="wheel_radius" value="0.065"/>
+    <xacro:property name="wheel_thickness" value="0.054"/>
     <xacro:property name="wheel_mass" value="0.05"/>
-    <xacro:property name="wheel_offset_x" value="0.25"/>
-    <xacro:property name="wheel_offset_y" value="0.115"/>
-    <xacro:property name="wheel_offset_z" value="0.0325"/>
+    <xacro:property name="wheel_offset_x" value="0.0"/>
+    <xacro:property name="wheel_offset_y" value="0.150"/>
+    <xacro:property name="wheel_offset_z" value="0.015"/>
     <material name="white">
         <color rgba="1 1 1 1" />
@@ -34,9 +34,9 @@
         <parent link="base_footprint"/>
         <child link="base_link"/>
-        <origin xyz="0 0 ${wheel_radius}"/>
+        <origin xyz="0 0 ${wheel_radius - 0.015}"/>
     </joint>
     <link name="base_link">
         <visual>
-            <origin xyz="${-chassis_length/2 + 0.05} 0 0"/>
+            <origin xyz="0 0 ${chassis_height/2}"/>
             <geometry>
                 <box size="${chassis_length} ${chassis_width} ${chassis_height}"/>
@@ -45,5 +45,5 @@
         </visual>
         <collision>
-            <origin xyz="${chassis_length/2} 0 ${chassis_height/2}"/>
+            <origin xyz="0 0 ${chassis_height/2}"/>
             <geometry>
                 <box size="${chassis_length} ${chassis_width} ${chassis_height}"/>
@@ -51,5 +51,5 @@
         </collision>
         <xacro:inertial_box mass="0.5" x="${chassis_length}" y="${chassis_width}" z="${chassis_height}">
-            <origin xyz="${chassis_length/2} 0 ${chassis_height/2}" rpy="0 0 0"/>
+            <origin xyz="0 0 ${chassis_height/2}" rpy="0 0 0"/>
         </xacro:inertial_box>
     </link>
@@ -61,5 +61,5 @@
         <parent link="base_link"/>
         <child link="left_wheel"/>
-        <origin xyz="0 ${wheel_offset_y} 0" rpy="-${pi/2} 0 0" />
+        <origin xyz="0 ${wheel_offset_y} ${wheel_offset_z}" rpy="-${pi/2} 0 0" />
         <axis xyz="0 0 1"/>
     </joint>
@@ -83,37 +83,9 @@
         <material>Gazebo/Blue</material>
     </gazebo>
-<!-- REAR LEFT WHEEL LINK -->
-    <joint name="rear_left_wheel_joint" type="fixed">
-        <parent link="base_link"/>
-        <child link="rear_left_wheel"/>
-        <origin xyz="-0.15 ${wheel_offset_y} 0" rpy="-${pi/2} 0 0" />
-        <axis xyz="0 0 1"/>
-    </joint>
-    <link name="rear_left_wheel">
-        <visual>
-            <geometry>
-                <cylinder radius="${wheel_radius}" length="${wheel_thickness}"/>
-            </geometry>
-            <material name="blue"/>
-        </visual>
-        <collision>
-            <geometry>
-                <sphere radius="${wheel_radius}"/>
-            </geometry>
-        </collision>
-        <xacro:inertial_cylinder mass="${wheel_mass}" length="${wheel_thickness}" radius="${wheel_radius}">
-            <origin xyz="0 0 0" rpy="0 0 0"/>
-        </xacro:inertial_cylinder>
-    </link>
-    <gazebo reference="rear_left_wheel">
-        <material>Gazebo/Blue</material>
-        <mu1 value="0.001"/>
-        <mu2 value="0.001"/>
-    </gazebo>
     <!-- RIGHT WHEEL LINK -->
     <joint name="right_wheel_joint" type="continuous">
         <parent link="base_link"/>
         <child link="right_wheel"/>
-        <origin xyz="0 ${-wheel_offset_y} 0" rpy="${pi/2} 0 0" />
+        <origin xyz="0 ${-wheel_offset_y} ${wheel_offset_z}" rpy="${pi/2} 0 0" />
         <axis xyz="0 0 -1"/>
     </joint>
@@ -137,21 +109,21 @@
         <material>Gazebo/Blue</material>
     </gazebo>
-    <!-- REAR RIGHT WHEEL LINK -->
-    <joint name="rear_right_wheel_joint" type="fixed">
+    <!-- REAR CASTER WHEEL -->
+    <joint name="rear_caster_wheel_joint" type="fixed">
         <parent link="base_link"/>
-        <child link="rear_right_wheel"/>
-        <origin xyz="-0.15 ${-wheel_offset_y} 0" rpy="${pi/2} 0 0" />
-        <axis xyz="0 0 -1"/>
+        <child link="rear_caster_wheel"/>
+        <origin xyz="-0.110 -0.10 -${wheel_radius - 0.0128 - 0.015}" rpy="${pi/2} 0 0" />
+        <axis xyz="0 0 0"/>
     </joint>
-    <link name="rear_right_wheel">
+    <link name="rear_caster_wheel">
         <visual>
             <geometry>
-                <cylinder radius="${wheel_radius}" length="${wheel_thickness}"/>
+                <cylinder radius="0.0128" length="0.0128"/>
             </geometry>
-            <material name="blue"/>
+            <material name="white"/>
         </visual>
         <collision>
             <geometry>
-                <sphere radius="${wheel_radius}"/>
+                <sphere radius="0.0128"/>
             </geometry>
         </collision>
@@ -160,5 +132,61 @@
         </xacro:inertial_cylinder>
     </link>
-    <gazebo reference="rear_right_wheel">
+    <gazebo reference="rear_caster_wheel">
+        <material>Gazebo/Blue</material>
+        <mu1 value="0.001"/>
+        <mu2 value="0.001"/>
+    </gazebo>
+    <!-- REAR CASTER WHEEL2 -->
+    <joint name="rear_caster_wheel2_joint" type="fixed">
+        <parent link="base_link"/>
+        <child link="rear_caster_wheel2"/>
+        <origin xyz="-0.110 0.10 -${wheel_radius - 0.0128 - 0.015}" rpy="${pi/2} 0 0" />
+        <axis xyz="0 0 0"/>
+    </joint>
+    <link name="rear_caster_wheel2">
+        <visual>
+            <geometry>
+                <cylinder radius="0.0128" length="0.0128"/>
+            </geometry>
+            <material name="white"/>
+        </visual>
+        <collision>
+            <geometry>
+                <sphere radius="0.0128"/>
+            </geometry>
+        </collision>
+        <xacro:inertial_cylinder mass="${wheel_mass}" length="${wheel_thickness}" radius="${wheel_radius}">
+            <origin xyz="0 0 0" rpy="0 0 0"/>
+        </xacro:inertial_cylinder>
+    </link>
+    <gazebo reference="rear_caster_wheel2">
+        <material>Gazebo/Blue</material>
+        <mu1 value="0.001"/>
+        <mu2 value="0.001"/>
+    </gazebo>
+    <!-- FRONT CASTER WHEEL -->
+    <joint name="front_caster_wheel_joint" type="fixed">
+        <parent link="base_link"/>
+        <child link="front_caster_wheel"/>
+        <origin xyz="0.110 0 -${wheel_radius - 0.0128 - 0.015}" rpy="${pi/2} 0 0" />
+        <axis xyz="0 0 0"/>
+    </joint>
+    <link name="front_caster_wheel">
+        <visual>
+            <geometry>
+                <cylinder radius="0.0128" length="0.0128"/>
+            </geometry>
+            <material name="white"/>
+        </visual>
+        <collision>
+            <geometry>
+                <sphere radius="0.0128"/>
+            </geometry>
+        </collision>
+        <xacro:inertial_cylinder mass="${wheel_mass}" length="${wheel_thickness}" radius="${wheel_radius}">
+            <origin xyz="0 0 0" rpy="0 0 0"/>
+        </xacro:inertial_cylinder>
+    </link>
+    <gazebo reference="front_caster_wheel">
         <material>Gazebo/Blue</material>
         <mu1 value="0.001"/>

File: lidarbot_description/urdf/ros2_control.xacro (robot description, xacro)
@@ -8,5 +8,5 @@
           <param name='left_wheel_name'>left_wheel_joint</param>
           <param name='right_wheel_name'>right_wheel_joint</param>
-          <param name='enc_ticks_per_rev'>1865</param>
+          <param name='enc_ticks_per_rev'>1888</param>
           <param name='loop_rate'>20.0</param>
       </hardware>
